File: KiCad/WristModule.kicad_pcb (KiCad board)
At the start: 2 copper layers, 40 x 55 mm, 79 parts, among them J1 USB_B_Micro, J2 Conn_01x22, J3 Conn_01x22, Q1 MUN5211DW1, SW1 SW_Push, T1 PBSS5330PAS, U1 ESP32-PICO-D4, U10 DRV2605LDGS, U11 MAX7358EUGT, U12 CD4051B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

Commit message: Add files via upload
Routing:
- net GND: track 294.0 -> 348.7 mm
Changed lines of the file:
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@@
     (thickness 1.6)
     (drawings 6)
-    (tracks 1405)
+    (tracks 1409)
     (zones 0)
     (modules 79)
@@
     (visible_elements 7FFDFFFF)
     (pcbplotparams
-      (layerselection 0x010f0_ffffffff)
+      (layerselection 0x3ffff_ffffffff)
       (usegerberextensions true)
       (usegerberattributes false)
@@
       (padsonsilk false)
       (subtractmaskfromsilk true)
-      (outputformat 1)
+      (outputformat 4)
       (mirror false)
       (drillshape 0)
@@
     (pad 49 smd rect (at 0 0 225) (size 5.3 5.3) (layers F.Cu F.Mask)
       (net 2 GND))
-    (pad "" smd roundrect (at -1.98 -1.98 225) (size 1.07 1.07) (layers F.Paste) (roundrect_rratio 0.233645))
-    (pad "" smd roundrect (at -1.98 -0.66 225) (size 1.07 1.07) (layers F.Paste) (roundrect_rratio 0.233645))
-    (pad "" smd roundrect (at -1.98 0.66 225) (size 1.07 1.07) (layers F.Paste) (roundrect_rratio 0.233645))
-    (pad "" smd roundrect (at -1.98 1.98 225) (size 1.07 1.07) (layers F.Paste) (roundrect_rratio 0.233645))
-    (pad "" smd roundrect (at -0.66 -1.98 225) (size 1.07 1.07) (layers F.Paste) (roundrect_rratio 0.233645))
-    (pad "" smd roundrect (at -0.66 -0.66 225) (size 1.07 1.07) (layers F.Paste) (roundrect_rratio 0.233645))
-    (pad "" smd roundrect (at -0.66 0.66 225) (size 1.07 1.07) (layers F.Paste) (roundrect_rratio 0.233645))
-    (pad "" smd roundrect (at -0.66 1.98 225) (size 1.07 1.07) (layers F.Paste) (roundrect_rratio 0.233645))
-    (pad "" smd roundrect (at 0.66 -1.98 225) (size 1.07 1.07) (layers F.Paste) (roundrect_rratio 0.233645))
-    (pad "" smd roundrect (at 0.66 -0.66 225) (size 1.07 1.07) (layers F.Paste) (roundrect_rratio 0.233645))
-    (pad "" smd roundrect (at 0.66 0.66 225) (size 1.07 1.07) (layers F.Paste) (roundrect_rratio 0.233645))
-    (pad "" smd roundrect (at 0.66 1.98 225) (size 1.07 1.07) (layers F.Paste) (roundrect_rratio 0.233645))
-    (pad "" smd roundrect (at 1.98 -1.98 225) (size 1.07 1.07) (layers F.Paste) (roundrect_rratio 0.233645))
-    (pad "" smd roundrect (at 1.98 -0.66 225) (size 1.07 1.07) (layers F.Paste) (roundrect_rratio 0.233645))
-    (pad "" smd roundrect (at 1.98 0.66 225) (size 1.07 1.07) (layers F.Paste) (roundrect_rratio 0.233645))
-    (pad "" smd roundrect (at 1.98 1.98 225) (size 1.07 1.07) (layers F.Paste) (roundrect_rratio 0.233645))
+    (pad "" smd roundrect (at -1.98 -1.98 225) (size 1.07 1.07) (layers F.Paste) (roundrect_rratio 0.2336448598130841))
+    (pad "" smd roundrect (at -1.98 -0.66 225) (size 1.07 1.07) (layers F.Paste) (roundrect_rratio 0.2336448598130841))
+    (pad "" smd roundrect (at -1.98 0.66 225) (size 1.07 1.07) (layers F.Paste) (roundrect_rratio 0.2336448598130841))
+    (pad "" smd roundrect (at -1.98 1.98 225) (size 1.07 1.07) (layers F.Paste) (roundrect_rratio 0.2336448598130841))
+    (pad "" smd roundrect (at -0.66 -1.98 225) (size 1.07 1.07) (layers F.Paste) (roundrect_rratio 0.2336448598130841))
+    (pad "" smd roundrect (at -0.66 -0.66 225) (size 1.07 1.07) (layers F.Paste) (roundrect_rratio 0.2336448598130841))
+    (pad "" smd roundrect (at -0.66 0.66 225) (size 1.07 1.07) (layers F.Paste) (roundrect_rratio 0.2336448598130841))
+    (pad "" smd roundrect (at -0.66 1.98 225) (size 1.07 1.07) (layers F.Paste) (roundrect_rratio 0.2336448598130841))
+    (pad "" smd roundrect (at 0.66 -1.98 225) (size 1.07 1.07) (layers F.Paste) (roundrect_rratio 0.2336448598130841))
+    (pad "" smd roundrect (at 0.66 -0.66 225) (size 1.07 1.07) (layers F.Paste) (roundrect_rratio 0.2336448598130841))
+    (pad "" smd roundrect (at 0.66 0.66 225) (size 1.07 1.07) (layers F.Paste) (roundrect_rratio 0.2336448598130841))
+    (pad "" smd roundrect (at 0.66 1.98 225) (size 1.07 1.07) (layers F.Paste) (roundrect_rratio 0.2336448598130841))
+    (pad "" smd roundrect (at 1.98 -1.98 225) (size 1.07 1.07) (layers F.Paste) (roundrect_rratio 0.2336448598130841))
+    (pad "" smd roundrect (at 1.98 -0.66 225) (size 1.07 1.07) (layers F.Paste) (roundrect_rratio 0.2336448598130841))
+    (pad "" smd roundrect (at 1.98 0.66 225) (size 1.07 1.07) (layers F.Paste) (roundrect_rratio 0.2336448598130841))
+    (pad "" smd roundrect (at 1.98 1.98 225) (size 1.07 1.07) (layers F.Paste) (roundrect_rratio 0.2336448598130841))
     (model ${KISYS3DMOD}/Package_DFN_QFN.3dshapes/QFN-48-1EP_7x7mm_P0.5mm_EP5.3x5.3mm.wrl
       (at (xyz 0 0 0))
@@
   (segment (start 142.175 52.7625) (end 143.7375 51.2) (width 0.25) (layer F.Cu) (net 2))
   (segment (start 142.175 53.05) (end 142.175 52.7625) (width 0.25) (layer F.Cu) (net 2))
+  (segment (start 174.64999 31.5) (end 173.3 31.5) (width 0.25) (layer F.Cu) (net 2))
+  (segment (start 174.64999 77.6) (end 174.64999 31.5) (width 0.25) (layer F.Cu) (net 2))
+  (segment (start 174.62499 77.625) (end 174.64999 77.6) (width 0.25) (layer F.Cu) (net 2))
+  (segment (start 167.425 77.625) (end 174.62499 77.625) (width 0.25) (layer F.Cu) (net 2))
   (segment (start 164.7 34.72) (end 164.7 35.7) (width 0.25) (layer F.Cu) (net 3))
   (segment (start 165.38 35.7) (end 165.43 35.75) (width 0.25) (layer F.Cu) (net 3))
